Commit message: tugas 2 kelompok robotika

File: urdf/macro.xacro (robot description, xacro)
@@ -23,5 +23,5 @@
     </xacro:macro>
     <xacro:macro name="joint_wheel" params="name child origin_xyz">
-      <joint name="${name}" type="continuous">
+      <joint name="${name}" type="fixed">
         <origin rpy="0 0 0" xyz="${origin_xyz}"/>
         <child link="${child}"/>

File: urdf/robot2roda.xacro (robot description, xacro)
@@ -26,5 +26,5 @@
     </visual>
     <!-- caster front -->
-    <collision name="caster_front_collision">
+<!-- <collision name="caster_front_collision">
       <origin rpy=" 0 0 0" xyz="0.35 0 -0.05"/>
       <geometry>
@@ -47,12 +47,69 @@
         <sphere radius="0.05"/>
       </geometry>
+    </visual> -->
+    </link>
+<!-- Create front right wheel -->
+  <link name="front_link_right_wheel">
+    <inertial>
+      <mass value="0.2"/>
+      <origin rpy="0 1.5707 1.5707" xyz="0 0 0"/>
+      <inertia ixx="0.00052666666" ixy="0" ixz="0" iyy="0.00052666666" iyz="0" izz="0.001"/>
+    </inertial>
+    <collision name="link_right_wheel_collision">
+      <origin rpy="0 1.5707 1.5707" xyz="0 0 0" />
+      <geometry>
+        <cylinder length="0.04" radius="0.1"/>
+      </geometry>
+    </collision>
+    <visual name="link_right_wheel_visual">
+      <origin rpy="0 1.5707 1.5707" xyz="0 0 0"/>
+      <geometry>
+        <cylinder length="0.04" radius="0.1"/>
+      </geometry>
     </visual>
-    </link>
+  </link>
+  <!--   Joint for right wheel  -->
+  <joint name="front_joint_right_wheel" type="continuous">
+    <origin rpy="0 0 0" xyz="0.15 0.15 0"/>
+    <child link="front_link_right_wheel" />
+    <parent link="link_chassis"/>
+    <axis rpy="0 0 0" xyz="0 1 0"/>
+    <limit effort="10000" velocity="1000"/>
+    <joint_properties damping="1.0" friction="1.0" />
+  </joint>
+<!-- Create front Left wheel -->
+<link name="front_link_left_wheel">
+    <inertial>
+      <mass value="0.2"/>
+      <origin rpy="0 1.5707 1.5707" xyz="0 0 0"/>
+      <inertia ixx="0.00052666666" ixy="0" ixz="0" iyy="0.00052666666" iyz="0" izz="0.001"/>
+    </inertial>
+    <collision name="link_left_wheel_collision">
+      <origin rpy="0 1.5707 1.5707" xyz="0 0 0" />
+      <geometry>
+        <cylinder length="0.04" radius="0.1"/>
+      </geometry>
+    </collision>
+    <visual name="link_left_wheel_visual">
+      <origin rpy="0 1.5707 1.5707" xyz="0 0 0"/>
+      <geometry>
+        <cylinder length="0.04" radius="0.1"/>
+      </geometry>
+    </visual>
+  </link>
+<joint name="joint_left_wheel" type="continuous">
+    <origin rpy="0 0 0" xyz="0.15 -0.15 0"/>
+    <child link="front_link_left_wheel" />
+    <parent link="link_chassis"/>
+    <axis rpy="0 0 0" xyz="0 1 0"/>
+    <limit effort="10000" velocity="1000"/>
+    <joint_properties damping="1.0" friction="1.0" />
+  </joint>
   <!-- Create wheel right -->
-   <xacro:link_wheel name="link_right_wheel" />
-   <xacro:joint_wheel name="joint_right_wheel"  child="link_right_wheel"  origin_xyz="-0.05 0.15 0"  />
+   <xacro:link_wheel name="back_link_right_wheel" />
+   <xacro:joint_wheel name="back_joint_right_wheel"  child="back_link_right_wheel"  origin_xyz="-0.15 0.15 0"  />
   <!-- Left Wheel link -->
-  <xacro:link_wheel name="link_left_wheel" />
-  <xacro:joint_wheel name="joint_left_wheel"   child="link_left_wheel"   origin_xyz="-0.05 -0.15 0"  />
+  <xacro:link_wheel name="back_link_left_wheel" />
+  <xacro:joint_wheel name="back_joint_left_wheel"   child="back_link_left_wheel"   origin_xyz="-0.15 -0.15 0"  />
 	<link name="sensor_laser">
     <inertial>
